File: board/sstv-backpack.kicad_pcb (KiCad board)
At the start: 2 copper layers, 38.1 x 63.5 mm, 10 parts, among them J1 Conn_01x03_Pin, SW1 SW_Push, SW2 SLW-1276864-4A-D, U1 ESP32-CAM

Commit message: Update silkscreen and gerbers
Parts:
- removed BAT IN: Conn_01x02_Pin, Connector_PinHeader_2.54mm:PinHeader_1x02_P2.54mm_Vertical
- added BAT_IN: Conn_01x02_Pin, Connector_PinHeader_2.54mm:PinHeader_1x02_P2.54mm_Vertical, F.Cu at (160.0, 124.5)
- added REF**: MountingHole_2.2mm_M2, MountingHole:MountingHole_2.2mm_M2, F.Cu at (175.3, 66.0)
- added REF**: MountingHole_2.2mm_M2, MountingHole:MountingHole_2.2mm_M2, F.Cu at (142.2, 66.0)
- added REF**: MountingHole_2.2mm_M2, MountingHole:MountingHole_2.2mm_M2, F.Cu at (175.3, 124.5)
- added REF**: MountingHole_2.2mm_M2, MountingHole:MountingHole_2.2mm_M2, F.Cu at (142.2, 124.5)
- moved J1 5.06 mm to (142.7, 85.1), turned to 180 degrees
Connections:
- J1 pad 1: /PTT -> GND
- J1 pad 3: GND -> /PTT
Other:
- outline, holes or cut-outs redrawn
- board text added: "+"
- board text added: "-"
- board text added: "1-GND"
- board text added: "2-AF OUT"
- board text added: "3-PTT"
- board text added: "J1"
