File: board/sstv-backpack.kicad_sch (KiCad schematic)
At the start: 10 parts, among them J1 Conn_01x03_Pin, J2 Conn_01x02_Pin, SW1 SW_Push, SW2 SLW-1276864-4A-D, U1 ESP32-CAM, U2 LP38693DT-5.0

Commit message: Update silkscreen and gerbers
Parts:
- renumbered J2 to BAT_IN, U2 to VR1
Connections:
- net GND: now also BAT_IN.1 (Pin_1), J1.1 (Pin_1); no longer BAT_IN.2 (Pin_2), J1.3 (Pin_3)
- net PTT: now also J1.3 (Pin_3); no longer J1.1 (Pin_1)
- net VIN: now also BAT_IN.2 (Pin_2); no longer BAT_IN.1 (Pin_1)
Other:
- moved on the sheet: J1
Changed lines of the file:
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@@
+	(wire
+		(pts
+			(xy 102.87 53.34) (xy 102.87 69.85)
+		)
+		(stroke
+			(width 0)
+			(type default)
+		)
+	)
 	(wire
 		(pts
@@
 	(wire
 		(pts
+			(xy 102.87 50.8) (xy 115.57 50.8)
+		)
+		(stroke
+			(width 0)
+			(type default)
+		)
+	)
+	(wire
+		(pts
 			(xy 163.83 69.85) (xy 179.07 69.85)
 		)
@@
 	(wire
 		(pts
+			(xy 143.51 125.73) (xy 165.1 125.73)
+		)
+		(stroke
+			(width 0)
+			(type default)
+		)
+	)
+	(wire
+		(pts
 			(xy 143.51 120.65) (xy 157.48 120.65)
 		)
@@
 	(wire
 		(pts
-			(xy 143.51 125.73) (xy 165.1 125.73)
-		)
-		(stroke
-			(width 0)
-			(type default)
-		)
-	)
-	(wire
-		(pts
-			(xy 102.87 50.8) (xy 115.57 50.8)
-		)
-		(stroke
-			(width 0)
-			(type default)
-		)
-	)
-	(wire
-		(pts
 			(xy 143.51 118.11) (xy 157.48 118.11)
-		)
-		(stroke
-			(width 0)
-			(type default)
-		)
-	)
-	(wire
-		(pts
-			(xy 102.87 53.34) (xy 102.87 69.85)
 		)
 		(stroke
@@
 		(dnp no)
 		(fields_autoplaced yes)
-		(property "Reference" "U2"
+		(property "Reference" "VR1"
 			(at 163.83 53.34 0)
 			(effects
@@
 			(project ""
 				(path "/29ea68c4-1664-4e2a-8c4b-cdbccd245911"
-					(reference "U2")
+					(reference "VR1")
 					(unit 1)
 				)
@@
 	(symbol
 		(lib_id "Connector:Conn_01x02_Pin")
-		(at 97.79 50.8 0)
-		(unit 1)
-		(exclude_from_sim no)
-		(in_bom yes)
-		(on_board yes)
-		(dnp no)
-		(fields_autoplaced yes)
-		(property "Reference" "J2"
-			(at 98.425 45.72 0)
+		(at 97.79 53.34 0)
+		(mirror x)
+		(unit 1)
+		(exclude_from_sim no)
+		(in_bom yes)
+		(on_board yes)
+		(dnp no)
+		(property "Reference" "BAT_IN"
+			(at 98.425 58.42 0)
 			(effects
 				(font
@@
 		)
 		(property "Value" "Conn_01x02_Pin"
-			(at 98.425 48.26 0)
+			(at 98.425 55.88 0)
 			(effects
 				(font
@@
 		)
 		(property "Footprint" "Connector_PinHeader_2.54mm:PinHeader_1x02_P2.54mm_Vertical"
-			(at 97.79 50.8 0)
+			(at 97.79 53.34 0)
 			(effects
 				(font
@@
 		)
 		(property "Datasheet" "~"
-			(at 97.79 50.8 0)
+			(at 97.79 53.34 0)
 			(effects
 				(font
@@
 		)
 		(property "Description" "Generic connector, single row, 01x02, script generated"
-			(at 97.79 50.8 0)
+			(at 97.79 53.34 0)
 			(effects
 				(font
@@
 			(project ""
 				(path "/29ea68c4-1664-4e2a-8c4b-cdbccd245911"
-					(reference "J2")
+					(reference "BAT_IN")
 					(unit 1)
 				)
@@
 	(symbol
 		(lib_id "Connector:Conn_01x03_Pin")
-		(at 162.56 118.11 180)
-		(unit 1)
-		(exclude_from_sim no)
-		(in_bom yes)
-		(on_board yes)
-		(dnp no)
-		(fields_autoplaced yes)
+		(at 162.56 118.11 0)
+		(mirror y)
+		(unit 1)
+		(exclude_from_sim no)
+		(in_bom yes)
+		(on_board yes)
+		(dnp no)
 		(property "Reference" "J1"
-			(at 163.83 116.8399 0)
+			(at 163.83 119.3801 0)
 			(effects
 				(font
@@
 		)
 		(property "Value" "Conn_01x03_Pin"
-			(at 163.83 119.3799 0)
-			(effects
-				(font
+			(at 163.83 116.8401 0)
+			(effects
+				(font
